Commit message: update robot.urdf

File: urdf/robot.urdf (robot description, URDF)
Before this commit: robot None, 7 links, 6 joints
Links:
- link base_link: geometry collision box size=0.4 0.307 0.102; visual mesh filename=../meshes/rover.stl
- link wheel_lb: geometry collision cylinder length=0.05 radius=0.05; visual mesh filename=../meshes/wheel_lb.stl
- link wheel_lf: geometry collision cylinder length=0.05 radius=0.05; visual mesh filename=../meshes/wheel_lf.stl
- link wheel_rb: geometry collision cylinder length=0.05 radius=0.05; visual mesh filename=../meshes/wheel_rb.stl
- link wheel_rf: geometry collision cylinder length=0.05 radius=0.05; visual mesh filename=../meshes/wheel_rf.stl
