Commit message: Update color values for materials in robot.xacro

File: urdf/robot.common.xacro (robot description, xacro)
@@ -42,11 +42,8 @@
 <!-- Color codes from https://gist.github.com/naoki-mizuno/5e63a13597d5c5fe817c1600b829595e, matches with Gazebo colors with the same name -->
 <material name="blue">
-    <color rgba="0.011764705882352941 0.2627450980392157 0.8745098039215686 1.0"/>
-</material>
-<material name="orangerover">
-    <color rgba="0.9764705882352941 0.45098039215686275 0.023529411764705882 1.0"/>
+    <color rgba="0.8 0.8 0.88 1.0"/>
 </material>
 <material name="darkgreyrover">
-    <color rgba="0.21176470588235294 0.21568627450980393 0.21568627450980393 1.0"/>
+    <color rgba="0.15 0.15 0.15 1.0"/>
 </material>
 </robot>

Commit message: Change material color from blue to lightgrey

File: urdf/robot.common.xacro (robot description, xacro)
@@ -41,5 +41,5 @@
 </xacro:macro>
 <!-- Color codes from https://gist.github.com/naoki-mizuno/5e63a13597d5c5fe817c1600b829595e, matches with Gazebo colors with the same name -->
-<material name="blue">
+<material name="lightgrey">
     <color rgba="0.8 0.8 0.88 1.0"/>
 </material>
