Commit message: rename KR0003 to KR003

File: urdf/robot.urdf.xacro (robot description, xacro)
@@ -1,7 +1,7 @@
 <?xml version="1.0" encoding="utf-8"?>
 <robot xmlns:xacro="http://ros.org/wiki/xacro">
-<xacro:include filename="$(find kr0003_description)/urdf/robot.common.xacro"/>
-<xacro:include filename="$(find kr0003_description)/urdf/robot.control.xacro"/>
-<xacro:property name="mesh_path" value="package://kr0003_description/meshes/"/>
+<xacro:include filename="$(find kr003_description)/urdf/robot.common.xacro"/>
+<xacro:include filename="$(find kr003_description)/urdf/robot.control.xacro"/>
+<xacro:property name="mesh_path" value="package://kr003_description/meshes/"/>
 <!-- **** LINKS **** -->
 <!-- BASE_FOOTPRINT -->

Commit message: Change material color from blue to lightgrey

File: urdf/robot.urdf.xacro (robot description, xacro)
@@ -14,5 +14,5 @@
       <mesh filename="${mesh_path}rover.stl" />
     </geometry>
-    <material name="blue"/>
+    <material name="lightgrey"/>
   </visual>
   <collision>
